Commit message: Fix robot contact under Bullet on 1F; add ground-truth checks
Ground-truth logging showed that on 1F the robot could not physically
turn under Bullet Featherstone. Its wheels turned at the commanded
rate, but the body rotated 0.000 of the commanded angle and moved 0.58
of the commanded distance, while odometry reported full motion. Every
1F sweep figure since the switch to Bullet therefore measured believed
pose only, and the docs now withdraw them.

Bare-floor experiments traced the fault to two contact settings:
- Bullet ignores <ode><mu> and sets friction once per link, so the
  lumped caster inherited the body's friction of 1.0. The caster is
  now a preserved fixed-joint link with ode and bullet friction 0.1.
- Bullet applies the torsional friction coefficient (SDF default 1.0)
  as spinning friction combined from both surfaces, locking yaw.
  Wheels, caster and the 1F ground plane now set it to 0.

With both, Bullet matches DART (spin, straight and arc all 1.000) and
DART is unaffected. In the 1F launch: real-time factor 1.00, LiDAR
alignment 99.4%, and the mesh still stops the robot 0.32 m from the wall.

DART cannot replace Bullet on 1F: it segfaults creating the wall mesh
shape with both its ODE and Bullet collision detectors.

The first logged sweep after the fix exposed three open problems,
recorded in CLAUDE.md and the README: base_footprint is 0.15 m ahead of
the wheel axle that odometry follows, the costmap robot_radius (0.27 m)
is smaller than the body (0.36 m), and AMCL does not correct the pose.

Adds to tools/sim_checks: gt_logger.py, gt_analyse.py, gt_supervisor.sh,
motion_test.py, bullet_friction_test.py, and DART world variants.

Co-Authored-By: Claude Opus 5 <noreply@anthropic.com>

File: my_robot_description/urdf/mobile_base_gazebo.xacro (robot description, xacro)
@@ -1,8 +1,41 @@
 <?xml version="1.0"?>
 <robot xmlns:xacro="http://www.ros.org/wiki/xacro">
+    <!-- Contact surfaces are written for both physics engines. 1F runs Bullet Featherstone,  -->
+    <!-- the other floors DART. Bullet ignores <ode><mu> (what <mu1>/<mu2> produce), sets     -->
+    <!-- friction once per link, and treats <torsional><coefficient> (SDF default 1.0) as     -->
+    <!-- spinning friction, which locked yaw completely. See the 1F motion tests of           -->
+    <!-- 15 September 2026 in spatial_maps/tools/sim_checks.                                  -->
+    <!-- Keep the caster as its own link. Lumped into base_footprint, its friction was       -->
+    <!-- overwritten by the body's default 1.0 under Bullet and the drive wheels slipped.    -->
+    <!-- (No colon-space in comments here. The launch files parse the URDF as YAML.)         -->
+    <gazebo reference="base_caster_wheel_joint">
+        <preserveFixedJoint>true</preserveFixedJoint>
+    </gazebo>
     <gazebo reference="caster_wheel_link">
-        <mu1 value="0.1"/>
-        <mu2 value="0.1"/>
+        <collision>
+            <surface>
+                <friction>
+                    <torsional><coefficient>0</coefficient></torsional>
+                    <ode><mu>0.1</mu><mu2>0.1</mu2></ode>
+                    <bullet><friction>0.1</friction><friction2>0.1</friction2><rolling_friction>0</rolling_friction></bullet>
+                </friction>
+            </surface>
+        </collision>
     </gazebo>
+    <!-- No torsional friction at the wheel contacts, or the robot cannot turn under Bullet. -->
+    <!-- The floor must also set it to 0, because Bullet combines wheel and floor values.    -->
+    <xacro:macro name="wheel_surface" params="prefix">
+        <gazebo reference="${prefix}_wheel_link">
+            <collision>
+                <surface>
+                    <friction>
+                        <torsional><coefficient>0</coefficient></torsional>
+                    </friction>
+                </surface>
+            </collision>
+        </gazebo>
+    </xacro:macro>
+    <xacro:wheel_surface prefix="left"/>
+    <xacro:wheel_surface prefix="right"/>
     <gazebo>
         <plugin filename="gz-sim-diff-drive-system" name="gz::sim::systems::DiffDrive">
