Commit message: Put base_footprint on the wheel axle; add footprint reachability study
The DiffDrive plugin's odometry follows the midpoint of the wheel axle,
but base_footprint sat 0.15 m ahead of it, under the body centre. Every
turn shifted the believed pose by 0.3*|sin(dheading/2)|, up to 0.30 m,
which let the robot clip a mapped wall corner in the first ground-truth
logged sweep. base_joint now places base_link 0.15 m ahead of
base_footprint, so the physical robot is unchanged.

Validated in the 1F launch: during a 10 rad spin the true base_footprint
moves 0.000 m (was 0.288 m) and matches odometry; straight driving is
1.002 of commanded; real-time factor 1.00; LiDAR alignment 99.0%. The
wall-contact test now reports a 0.47 m gap because the reference point
is 0.15 m further back; the body stops in the same place.

Note: the costmaps still use robot_radius 0.27 about base_footprint,
while the body now reaches 0.46 m ahead of it. Do not run sweeps until
the footprint is updated.

footprint_reachability.py is an offline study of which 1F sweep goals a
footprint can reach, under a circular planning model and an SE2 model
with in-place rotation only where it fits. With the current robot and
0.05 m padding, the circular model reaches 63 of 74 goals and the SE2
model 74 of 74. Control runs with larger footprints lose goals as
expected.

Co-Authored-By: Claude Opus 5 <noreply@anthropic.com>

File: my_robot_description/urdf/mobile_base.xacro (robot description, xacro)
@@ -59,8 +59,11 @@
         <xacro:sphere_inertia m="0.5" r="${wheel_radius / 2.0}" o_xyz="0 0 0" o_rpy="0 0 0"/>
     </link>
+    <!-- base_footprint sits on the midpoint of the wheel axle, which is the point the    -->
+    <!-- DiffDrive odometry follows. With base_footprint under the body centre instead,   -->
+    <!-- every turn shifted the believed pose by up to 0.30 m (15 September 2026).         -->
     <joint name="base_joint" type="fixed">
         <parent link="base_footprint"/>
         <child link="base_link"/>
-        <origin xyz="0 0 ${wheel_radius}" rpy="0 0 0"/>
+        <origin xyz="${base_length / 4.0} 0 ${wheel_radius}" rpy="0 0 0"/>
     </joint>
     <joint name="base_right_wheel_joint" type="continuous">
